Commit message: modified package location

File: urdf/red_robot.urdf (robot description, URDF)
Before this commit: robot red_robot, 36 links, 35 joints
Links:
- link AnkleCenter_L_Link: geometry collision mesh filename=package://red_description/meshes/AnkleCenter_L_Link.stl; visual mesh filename=package://red_description/meshes/AnkleCenter_L_Link.stl
- link AnkleCenter_R_Link: geometry visual mesh filename=package://red_description/meshes/AnkleCenter_R_Link.stl
- link AnkleRoll_L_Link: geometry collision mesh filename=package://red_description/meshes/AnkleRoll_L_Link.stl; visual mesh filename=package://red_description/meshes/AnkleRoll_L_Link.stl
- link AnkleRoll_R_Link: geometry collision mesh filename=package://red_description/meshes/AnkleRoll_R_Link.stl scale=1 1 1; visual mesh filename=package://red_description/meshes/AnkleRoll_R_Link.stl
- link Head: geometry collision mesh filename=package://red_description/meshes/head.stl; visual mesh filename=package://red_description/meshes/head.stl
- link HipCenter_L_Link: geometry visual mesh filename=package://red_description/meshes/HipCenter_L_Link.stl
- link HipCenter_R_Link: geometry visual mesh filename=package://red_description/meshes/HipCenter_R_Link.stl
- link HipRoll_L_Link: geometry visual mesh filename=package://red_description/meshes/HipRoll_L_Link.stl
- link HipRoll_R_link: geometry visual mesh filename=package://red_description/meshes/HipRoll_R_link.stl
- link Knee_L_Link: geometry collision mesh filename=package://red_description/meshes/Knee_L_Link.stl; visual mesh filename=package://red_description/meshes/Knee_L_Link.stl
- link Knee_R_Link: geometry visual mesh filename=package://red_description/meshes/Knee_R_Link.stl
- link L_armlink: geometry collision mesh filename=package://red_description/meshes/L_arm.stl; visual mesh filename=package://red_description/meshes/L_arm.stl
- link L_elbow: geometry collision mesh filename=package://red_description/meshes/L_elbow.stl; visual mesh filename=package://red_description/meshes/L_elbow.stl
- link L_forearm: geometry collision mesh filename=package://red_description/meshes/L_forearm.stl; visual mesh filename=package://red_description/meshes/L_forearm.stl
- link L_shoulder1: geometry collision mesh filename=package://red_description/meshes/L_shoulder1.stl; visual mesh filename=package://red_description/meshes/L_shoulder1.stl
- link L_shoulder2: geometry collision mesh filename=package://red_description/meshes/L_shoulder2.stl; visual mesh filename=package://red_description/meshes/L_shoulder2.stl
- link L_shoulder3: geometry collision mesh filename=package://red_description/meshes/L_shoulder3.stl; visual mesh filename=package://red_description/meshes/L_shoulder3.stl
- link L_wrist1: geometry collision mesh filename=package://red_description/meshes/L_wrist1.stl; visual mesh filename=package://red_description/meshes/L_wrist1.stl
- link L_wrist2: geometry collision mesh filename=package://red_description/meshes/L_wrist2.stl; visual mesh filename=package://red_description/meshes/L_wrist2.stl
- link Neck: geometry collision mesh filename=package://red_description/meshes/neck.stl; visual mesh filename=package://red_description/meshes/neck.stl
- link Pelvis_link: geometry collision mesh filename=package://red_description/meshes/Pelvis_link.stl; visual mesh filename=package://red_description/meshes/Pelvis_link.stl
- link R_armlink: geometry collision mesh filename=package://red_description/meshes/R_arm.stl; visual mesh filename=package://red_description/meshes/R_arm.stl
- link R_elbow: geometry collision mesh filename=package://red_description/meshes/R_elbow.stl; visual mesh filename=package://red_description/meshes/R_elbow.stl
- link R_forearm: geometry collision mesh filename=package://red_description/meshes/R_forearm.stl; visual mesh filename=package://red_description/meshes/R_forearm.stl
- link R_shoulder1: geometry collision mesh filename=package://red_description/meshes/R_shoulder1.stl; visual mesh filename=package://red_description/meshes/R_shoulder1.stl
- link R_shoulder2: geometry collision mesh filename=package://red_description/meshes/R_shoulder2.stl; visual mesh filename=package://red_description/meshes/R_shoulder2.stl
- link R_shoulder3: geometry collision mesh filename=package://red_description/meshes/R_shoulder3.stl; visual mesh filename=package://red_description/meshes/R_shoulder3.stl
- link R_wrist1: geometry collision mesh filename=package://red_description/meshes/R_wrist1.stl; visual mesh filename=package://red_description/meshes/R_wrist1.stl
- link R_wrist2: geometry collision mesh filename=package://red_description/meshes/R_wrist2.stl; visual mesh filename=package://red_description/meshes/R_wrist2.stl
- link Thigh_L_Link: geometry visual mesh filename=package://red_description/meshes/Thigh_L_Link.stl
- link Thigh_R_Link: geometry visual mesh filename=package://red_description/meshes/Thigh_R_Link.stl
- link Upperbody: geometry collision mesh filename=package://red_description/meshes/upperbody.stl; visual mesh filename=package://red_description/meshes/upperbody.stl
- link Waist1: geometry collision mesh filename=package://red_description/meshes/waist1.stl; visual mesh filename=package://red_description/meshes/waist1.stl
- link Waist2: geometry collision mesh filename=package://red_description/meshes/waist2.stl; visual mesh filename=package://red_description/meshes/waist2.stl
